Commit message: ycb exp

File: vbcpm_execution_system/data/models/robot/motoman.urdf (robot description, URDF)
Before this commit: robot sda10f, 33 links, 32 joints
Joints:
- joint left_inner_finger_joint: mimic joint=finger_joint multiplier=-1 offset=0 -> (none)
- joint left_inner_knuckle_joint: mimic joint=finger_joint multiplier=1 offset=0 -> (none)
- joint right_inner_finger_joint: limit lower=-0.8757 upper=0 effort=1000 velocity=2.0 -> (none); mimic joint=finger_joint multiplier=-1 offset=0 -> (none)
- joint right_inner_knuckle_joint: mimic joint=finger_joint multiplier=1 offset=0 -> (none)
- joint right_outer_knuckle_joint: mimic joint=finger_joint multiplier=1 offset=0 -> (none)
